File: examples/preamp/cad/tembr.sch (KiCad schematic (older format))
At the start: 60 parts, among them CON1 AVR-ISP-10, J1 CONN_01X02, J2 CONN_01X11, J3 CONN_01X03, J4 CONN_01X02, J5 CONN_01X03, J6 CONN_01X07, J7 CONN_01X02, J8 CONN_01X08, J9 CONN_01X08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

Commit message: Preamp schematic update kicad version
Parts:
- removed J2: CONN_01X11, Pin_Headers:Pin_Header_Straight_1x11_Pitch2.54mm, symbol CONN_01X11
- removed Q2: ., TO_SOT_Packages_THT:TO-92_Molded_Wide_Oval, symbol Q_NPN_BCE
- removed R1, R3: 20k*, Resistors_THT:R_Axial_DIN0207_L6.3mm_D2.5mm_P10.16mm_Horizontal, symbol R
- removed R11, R12: 3k, Resistors_THT:R_Axial_DIN0207_L6.3mm_D2.5mm_P10.16mm_Horizontal, symbol R
- removed R6, R7: 10k, Resistors_THT:R_Axial_DIN0207_L6.3mm_D2.5mm_P10.16mm_Horizontal, symbol R
- removed SW6: SW_Push_Dual, Buttons_Switches_THT:SW_PUSH_6mm, symbol SW_Push_Dual
- added J2: Conn_01x04, symbol Connector_Generic:Conn_01x04
- BT1: symbol Battery_Cell -> Device:Battery_Cell
- C1, C13, C15, C16, C18, C19, C20, C21, C22, C3, C6: symbol C_Small -> Device:C_Small
- C10, C11, C12, C14, C17, C23, C4, C5, C7, C8, C9: symbol CP_Small -> Device:CP_Small
- C2: symbol C_Small -> Device:CP_Small
- CON1: symbol AVR-ISP-10 -> Connector:AVR-ISP-10
- D1: symbol D -> Device:D
- J1, J4, J7: symbol CONN_01X02 -> Connector_Generic:Conn_01x02
- J3, J5: symbol CONN_01X03 -> Connector_Generic:Conn_01x03
- J6: symbol CONN_01X07 -> Connector_Generic:Conn_01x07
- J8, J9: symbol CONN_01X08 -> Connector_Generic:Conn_01x08
- Q1: symbol Q_NPN_BCE -> Device:Q_NPN_BCE
- R10, R2, R8, R9: symbol R -> Device:R
- R4, R5: value 100k -> 10k; symbol R -> Device:R
- SW1: symbol Rotary_Encoder -> Device:Rotary_Encoder_Switch
- SW2, SW3, SW4, SW5: symbol SW_Push_Dual -> Switch:SW_Push_Dual
- U1: footprint Housings_DIP:DIP-28_W7.62mm_LongPads -> Package_DIP:DIP-28_W7.62mm_LongPads; symbol ATMEGA8A-PU -> MCU_Microchip_ATmega:ATmega8A-PU
- U2: symbol DS1307+ -> Timer_RTC:DS1307ZN+
- U3: symbol LM7809CT -> Regulator_Linear:L7809
- U4: symbol TDA7313 -> tembr:TDA7313
- Y1: symbol Crystal -> Device:Crystal
Connections:
- net labels added: BTN3_MOSI, PowerBTN_MISO, SCK
- net labels removed: BL, BTN3/MISO, BTN4/SCK, Contr, D0, D1, D2, D3/MOSI, E, LED, RS, RW
- wire segments 213 -> 200
Other:
- moved on the sheet: BT1, CON1, Y1

Commit message: Start preamp PCB
Parts:
- BT1: footprint Battery_Holders:Keystone_1058_1x2032-CoinCell -> Battery:BatteryHolder_Keystone_103_1x20mm
- C1, C13, C15, C16, C18, C19, C2, C20, C21, C22, C3, C6: footprint Capacitors_THT:C_Rect_L9.0mm_W2.5mm_P7.50mm_MKT -> Capacitor_THT:C_Rect_L9.0mm_W2.5mm_P7.50mm_MKT
- C10, C11, C12, C14, C17, C23, C4, C5, C7, C8, C9: footprint Capacitors_THT:CP_Radial_D5.0mm_P2.50mm -> Capacitor_THT:CP_Radial_D5.0mm_P2.50mm
- CON1: footprint Connectors:IDC_Header_Straight_10pins -> Connector_IDC:IDC-Header_2x05_P2.54mm_Vertical
- D1: footprint Diodes_THT:D_T-1_P10.16mm_Horizontal -> Diode_THT:D_T-1_P10.16mm_Horizontal
- J1, J4, J7: footprint Pin_Headers:Pin_Header_Straight_1x02_Pitch2.54mm -> Connector_PinHeader_2.54mm:PinHeader_1x02_P2.54mm_Vertical
- J2: footprint (none) -> Connector_PinHeader_2.54mm:PinHeader_1x04_P2.54mm_Vertical
- J3, J5: footprint Pin_Headers:Pin_Header_Straight_1x03_Pitch2.54mm -> Connector_PinHeader_2.54mm:PinHeader_1x03_P2.54mm_Vertical
- J6: footprint Pin_Headers:Pin_Header_Straight_1x07_Pitch2.54mm -> Connector_PinHeader_2.00mm:PinHeader_1x07_P2.00mm_Vertical
- J8, J9: footprint Pin_Headers:Pin_Header_Straight_1x08_Pitch2.54mm -> Connector_PinHeader_2.54mm:PinHeader_1x08_P2.54mm_Vertical
- Q1: footprint TO_SOT_Packages_THT:TO-92_Molded_Wide_Oval -> Package_TO_SOT_THT:TO-92_HandSolder
- R10, R2, R4, R5, R8, R9: footprint Resistors_THT:R_Axial_DIN0207_L6.3mm_D2.5mm_P10.16mm_Horizontal -> Resistor_THT:R_Axial_DIN0207_L6.3mm_D2.5mm_P10.16mm_Horizontal
- SW1: footprint Potentiometers:Potentiometer_Alps_RK09K_Horizontal -> Rotary_Encoder:RotaryEncoder_Alps_EC11E-Switch_Vertical_H20mm
- SW2, SW3, SW4, SW5: footprint Buttons_Switches_THT:SW_PUSH_6mm -> Button_Switch_THT:SW_PUSH_6mm
- U2: footprint Housings_SOIC:SOIC-8_3.9x4.9mm_Pitch1.27mm -> Package_SO:SOIC-8_3.9x4.9mm_P1.27mm
- U3: footprint TO_SOT_Packages_THT:TO-220_Horizontal -> Package_TO_SOT_THT:TO-220-3_Horizontal_TabDown
- U4: footprint Housings_SOIC:SOIC-28W_7.5x17.9mm_Pitch1.27mm -> Package_SO:SOIC-28W_7.5x18.7mm_P1.27mm
- Y1: footprint Crystals:Crystal_AT310_d3.0mm_l10.0mm_Horizontal -> Crystal:Crystal_AT310_D3.0mm_L10.0mm_Horizontal
Connections:
- wire segments 200 -> 204
