File: examples/preamp/cad/preamp.sch (KiCad schematic (older format))
At the start: 52 parts, among them CON1 AVR-ISP-10, J1 CONN_01X02, J2 Conn_01x04, J3 CONN_01X03, J4 CONN_01X02, J5 CONN_01X03, J6 CONN_01X07, J7 CONN_01X02, J8 CONN_01X08, J9 CONN_01X08, Q1 ., SW1 Rotary_Encoder, SW2 SW_Push_Dual, SW3 SW_Push_Dual, SW4 SW_Push_Dual, SW5 SW_Push_Dual, U1 ATMEGA8A-PU, U2 DS1307+, U3 LM7809CT, U4 TDA7313, Y1 Crystal

Commit message: Rename kicad project
Parts:
- removed J6: CONN_01X07, Connector_PinHeader_2.00mm:PinHeader_1x07_P2.00mm_Vertical, symbol Connector_Generic:Conn_01x07
- added J10, J11, J6: Conn_01x03, Connector_PinHeader_2.54mm:PinHeader_1x03_P2.54mm_Vertical, symbol Connector_Generic:Conn_01x03
- U4: symbol tembr:TDA7313 -> preamp:TDA7313
Connections:
- wire segments 204 -> 219
Changed lines of the file:
@@
 EESchema Schematic File Version 4
-LIBS:tembr-cache
+LIBS:preamp-cache
 EELAYER 30 0
 EELAYER END
@@
 +9V
 $Comp
-L tembr:TDA7313 U4
+L preamp:TDA7313 U4
 U 1 1 5A02EE35
 P 12100 6350
@@
 $EndComp
 $Comp
-L Connector_Generic:Conn_01x07 J6
-U 1 1 5A035898
-P 10100 5550
-F 0 "J6" H 10100 5950 50  0000 C CNN
-F 1 "CONN_01X07" V 10200 5550 50  0000 C CNN
-F 2 "Connector_PinHeader_2.00mm:PinHeader_1x07_P2.00mm_Vertical" H 10100 5550 50  0001 C CNN
-F 3 "~" H 10100 5550 50  0001 C CNN
-	1    10100 5550
-	-1   0    0    1
-$EndComp
-$Comp
 L Connector_Generic:Conn_01x03 J5
 U 1 1 5A0359FA
@@
 L power:GNDA #PWR011
 U 1 1 5A036037
-P 10300 6050
-F 0 "#PWR011" H 10300 5800 50  0001 C CNN
-F 1 "GNDA" H 10300 5900 50  0000 C CNN
-F 2 "" H 10300 6050 50  0001 C CNN
-F 3 "" H 10300 6050 50  0001 C CNN
-	1    10300 6050
+P 10000 6300
+F 0 "#PWR011" H 10000 6050 50  0001 C CNN
+F 1 "GNDA" H 10000 6150 50  0000 C CNN
+F 2 "" H 10000 6300 50  0001 C CNN
+F 3 "" H 10000 6300 50  0001 C CNN
+	1    10000 6300
 	1    0    0    -1
 $EndComp
@@
 	10300 5250 10600 5250
 Wire Wire Line
-	10300 5350 10850 5350
-Wire Wire Line
-	10300 5450 10600 5450
-Wire Wire Line
 	10600 5450 10600 5550
 Wire Wire Line
-	10300 5550 10550 5550
-Wire Wire Line
 	10550 5550 10550 5650
 Wire Wire Line
 	10550 5650 10850 5650
 Wire Wire Line
-	10300 5650 10500 5650
-Wire Wire Line
 	10500 5650 10500 5850
 Wire Wire Line
 	10500 5850 10600 5850
 Wire Wire Line
-	10300 5750 10450 5750
-Wire Wire Line
 	10450 5750 10450 5950
 Wire Wire Line
 	10450 5950 10900 5950
-Wire Wire Line
-	10300 5850 10300 6050
 Wire Wire Line
 	13400 5450 13400 5600
@@
 Wire Wire Line
 	5150 3450 6100 3450
+$Comp
+L Connector_Generic:Conn_01x03 J6
+U 1 1 5DD651FA
+P 9750 5200
+F 0 "J6" H 9668 4875 50  0000 C CNN
+F 1 "Conn_01x03" H 9668 4966 50  0000 C CNN
+F 2 "Connector_PinHeader_2.54mm:PinHeader_1x03_P2.54mm_Vertical" H 9750 5200 50  0001 C CNN
+F 3 "~" H 9750 5200 50  0001 C CNN
+	1    9750 5200
+	-1   0    0    1
+$EndComp
+$Comp
+L Connector_Generic:Conn_01x03 J10
+U 1 1 5DD66517
+P 9750 5550
+F 0 "J10" H 9668 5225 50  0000 C CNN
+F 1 "Conn_01x03" H 9668 5316 50  0000 C CNN
+F 2 "Connector_PinHeader_2.54mm:PinHeader_1x03_P2.54mm_Vertical" H 9750 5550 50  0001 C CNN
+F 3 "~" H 9750 5550 50  0001 C CNN
+	1    9750 5550
+	-1   0    0    1
+$EndComp
+$Comp
+L Connector_Generic:Conn_01x03 J11
+U 1 1 5DD66C0D
+P 9750 5900
+F 0 "J11" H 9668 5575 50  0000 C CNN
+F 1 "Conn_01x03" H 9668 5666 50  0000 C CNN
+F 2 "Connector_PinHeader_2.54mm:PinHeader_1x03_P2.54mm_Vertical" H 9750 5900 50  0001 C CNN
+F 3 "~" H 9750 5900 50  0001 C CNN
+	1    9750 5900
+	-1   0    0    1
+$EndComp
+Wire Wire Line
+	9950 5100 10300 5100
+Wire Wire Line
+	10300 5100 10300 5250
+Wire Wire Line
+	9950 5200 10250 5200
+Wire Wire Line
+	10250 5200 10250 5350
+Wire Wire Line
+	10250 5350 10850 5350
+Wire Wire Line
+	9950 5450 10600 5450
+Wire Wire Line
+	9950 5550 10550 5550
+Wire Wire Line
+	9950 5800 10050 5800
+Wire Wire Line
+	10050 5800 10050 5650
+Wire Wire Line
+	10050 5650 10500 5650
+Wire Wire Line
+	9950 5900 10150 5900
+Wire Wire Line
+	10150 5900 10150 5750
+Wire Wire Line
+	10150 5750 10450 5750
+Wire Wire Line
+	9950 6000 10000 6000
+Wire Wire Line
+	10000 6000 10000 6300
+Wire Wire Line
+	10000 6000 10000 5650
+Wire Wire Line
+	10000 5650 9950 5650
+Connection ~ 10000 6000
+Wire Wire Line
+	10000 5650 10000 5300
+Wire Wire Line
+	10000 5300 9950 5300
+Connection ~ 10000 5650
+Entry Wire Line
+	6100 2950 6200 3050
+Wire Wire Line
+	6100 2950 5150 2950
+Entry Wire Line
+	6100 3050 6200 3150
+Wire Wire Line
+	6100 3050 5150 3050
 Wire Bus Line
 	6200 1900 8400 1900
@@
 Wire Bus Line
 	6200 1900 6200 9200
+Text Label 5700 2950 0    60   ~ 0
+LEFT
+Text Label 5700 3050 0    60   ~ 0
+RIGHT
 $EndSCHEMATC

Commit message: Update kicad project
Changed lines of the file:
@@
 EESchema Schematic File Version 4
-LIBS:preamp-cache
 EELAYER 30 0
 EELAYER END
@@
 	6100 3250 6200 3350
 Entry Wire Line
-	6100 2750 6200 2850
-Entry Wire Line
-	6100 2850 6200 2950
+	6100 3850 6200 3950
+Entry Wire Line
+	6100 3950 6200 4050
 Text Label 5700 3650 0    60   ~ 0
 IRint
@@
 	1    0    0    -1
 $EndComp
-Text Label 5700 2750 0    60   ~ 0
+Text Label 5700 3850 0    60   ~ 0
 ENC0
-Text Label 5700 2850 0    60   ~ 0
+Text Label 5700 3950 0    60   ~ 0
 ENC1
 Entry Wire Line
@@
 	5150 2550 6100 2550
 Wire Wire Line
-	5150 2750 6100 2750
-Wire Wire Line
-	5150 2850 6100 2850
+	5150 3850 6100 3850
+Wire Wire Line
+	5150 3950 6100 3950
 Wire Wire Line
 	5150 3150 6100 3150
@@
 Wire Wire Line
 	6100 3050 5150 3050
+Text Label 5700 2950 0    60   ~ 0
+LEFT
+Text Label 5700 3050 0    60   ~ 0
+RIGHT
 Wire Bus Line
 	6200 1900 8400 1900
@@
 Wire Bus Line
 	6200 1900 6200 9200
-Text Label 5700 2950 0    60   ~ 0
-LEFT
-Text Label 5700 3050 0    60   ~ 0
-RIGHT
 $EndSCHEMATC

Commit message: Update preamp scheme
Parts:
- R10, R8: value 5.5k -> 5.6k
Changed lines of the file:
@@
 P 13850 6900
 F 0 "R8" V 13930 6900 50  0000 C CNN
-F 1 "5.5k" V 13850 6900 50  0000 C CNN
+F 1 "5.6k" V 13850 6900 50  0000 C CNN
 F 2 "Resistor_THT:R_Axial_DIN0207_L6.3mm_D2.5mm_P10.16mm_Horizontal" V 13780 6900 50  0001 C CNN
 F 3 "~" H 13850 6900 50  0001 C CNN
@@
 P 13850 7200
 F 0 "R10" V 13930 7200 50  0000 C CNN
-F 1 "5.5k" V 13850 7200 50  0000 C CNN
+F 1 "5.6k" V 13850 7200 50  0000 C CNN
 F 2 "Resistor_THT:R_Axial_DIN0207_L6.3mm_D2.5mm_P10.16mm_Horizontal" V 13780 7200 50  0001 C CNN
 F 3 "~" H 13850 7200 50  0001 C CNN
@@
 Entry Wire Line
 	8400 2500 8500 2400
-Text Label 8550 2600 0    60   ~ 0
-SCL
 Wire Wire Line
 	8500 2600 8800 2600
 Entry Wire Line
 	8400 2700 8500 2600
-Text Label 8550 2700 0    60   ~ 0
-SDA
 Wire Wire Line
 	8500 2700 8800 2700
@@
 Wire Bus Line
 	6200 1900 6200 9200
+Text Label 8550 2600 0    50   ~ 0
+SDA
+Text Label 8550 2700 0    50   ~ 0
+SCL
 $EndSCHEMATC

Commit message: Update preamp scheme
Parts:
- removed D1: D, Diode_THT:D_T-1_P10.16mm_Horizontal, symbol Device:D
- removed J1, J7: CONN_01X02, Connector_PinHeader_2.54mm:PinHeader_1x02_P2.54mm_Vertical, symbol Connector_Generic:Conn_01x02
- removed J8, J9: CONN_01X08, Connector_PinHeader_2.54mm:PinHeader_1x08_P2.54mm_Vertical, symbol Connector_Generic:Conn_01x08
- removed SW1: Rotary_Encoder, Rotary_Encoder:RotaryEncoder_Alps_EC11E-Switch_Vertical_H20mm, symbol Device:Rotary_Encoder_Switch
- removed SW2, SW3, SW4, SW5: SW_Push_Dual, Button_Switch_THT:SW_PUSH_6mm, symbol Switch:SW_Push_Dual
- added J1: Conn_01x04, Connector_PinHeader_2.54mm:PinHeader_1x04_P2.54mm_Vertical, symbol Connector_Generic:Conn_01x04
- added J2, J3, J4, J5, J6: Conn_01x03, Connector_PinHeader_2.54mm:PinHeader_1x03_P2.54mm_Vertical, symbol Connector_Generic:Conn_01x03
- added Q2: ., Package_TO_SOT_THT:TO-92_HandSolder, symbol Device:Q_NPN_BCE
- added R2: 10k, Resistor_THT:R_Axial_DIN0207_L6.3mm_D2.5mm_P10.16mm_Horizontal, symbol Device:R
- R1: renamed from R9; value 3k -> 10k
- renumbered C2 to C1, C14 to C10, C17 to C11, C4 to C12, C5 to C13, C23 to C14, C6 to C15, C13 to C16, C16 to C17, C19 to C18, C21 to C19, C1 to C2, C15 to C20, C18 to C21, C20 to C22, C22 to C23, C7 to C3, C9 to C4, C11 to C5, C8 to C6, C10 to C7, C3 to C8, C12 to C9, J4 to J12, J5 to J13, J2 to J7, J3 to J8, J6 to J9, R4 to R3, R5 to R4, R2 to R5, R8 to R6, R10 to R7
Connections:
- net labels added: C945, CancelBtn, DownBtn, Encoder, LCD, Power&Relay, PowerBtn, PowerLED, StandBy, UpBtn
- net labels removed: A1_GND
- wire segments 219 -> 205
Other:
- note added: "30mA max"

Commit message: Add 3 Input buttons
Parts:
- removed J2: Conn_01x03, Connector_PinHeader_2.54mm:PinHeader_1x03_P2.54mm_Vertical, symbol Connector_Generic:Conn_01x03
- added J14, J15, J16, J2: Conn_01x04, Connector_PinHeader_2.54mm:PinHeader_1x04_P2.54mm_Vertical, symbol Connector_Generic:Conn_01x04
Connections:
- net labels added: Input1Btn, Input1Led, Input2Btn, Input2Led, Input3Btn, Input3Led
- wire segments 205 -> 221

Commit message: Update preamp scheme
Parts:
- removed J3, J4, J5: Conn_01x03, Connector_PinHeader_2.54mm:PinHeader_1x03_P2.54mm_Vertical, symbol Connector_Generic:Conn_01x03
- added J3, J4, J5: Conn_01x04, Connector_JST:JST_EH_B4B-EH-A_1x04_P2.50mm_Vertical, symbol Connector_Generic:Conn_01x04
- J1, J2: footprint Connector_PinHeader_2.54mm:PinHeader_1x04_P2.54mm_Vertical -> Connector_JST:JST_EH_B4B-EH-A_1x04_P2.50mm_Vertical
- J10: renamed from J7; footprint Connector_PinHeader_2.54mm:PinHeader_1x04_P2.54mm_Vertical -> Connector_JST:JST_EH_B4B-EH-A_1x04_P2.50mm_Vertical
- J11: renamed from J8; footprint Connector_PinHeader_2.54mm:PinHeader_1x03_P2.54mm_Vertical -> Connector_JST:JST_EH_B3B-EH-A_1x03_P2.50mm_Vertical
- J12: renamed from J9; footprint Connector_PinHeader_2.54mm:PinHeader_1x03_P2.54mm_Vertical -> TerminalBlock_Phoenix:TerminalBlock_Phoenix_MKDS-3-3-5.08_1x03_P5.08mm_Horizontal
- J13: renamed from J10; footprint Connector_PinHeader_2.54mm:PinHeader_1x03_P2.54mm_Vertical -> TerminalBlock_Phoenix:TerminalBlock_Phoenix_MKDS-3-3-5.08_1x03_P5.08mm_Horizontal
- J14: renamed from J11; footprint Connector_PinHeader_2.54mm:PinHeader_1x03_P2.54mm_Vertical -> TerminalBlock_Phoenix:TerminalBlock_Phoenix_MKDS-3-3-5.08_1x03_P5.08mm_Horizontal
- J15: renamed from J12; footprint Connector_PinHeader_2.54mm:PinHeader_1x02_P2.54mm_Vertical -> Connector_JST:JST_EH_B3B-EH-A_1x03_P2.50mm_Vertical
- J16: renamed from J13; footprint Connector_PinHeader_2.54mm:PinHeader_1x03_P2.54mm_Vertical -> TerminalBlock_Phoenix:TerminalBlock_Phoenix_MKDS-3-3-5.08_1x03_P5.08mm_Horizontal
- J6: renamed from J14; footprint Connector_PinHeader_2.54mm:PinHeader_1x04_P2.54mm_Vertical -> Connector_JST:JST_EH_B4B-EH-A_1x04_P2.50mm_Vertical
- J7: renamed from J15; footprint Connector_PinHeader_2.54mm:PinHeader_1x04_P2.54mm_Vertical -> Connector_JST:JST_EH_B4B-EH-A_1x04_P2.50mm_Vertical
- J8: renamed from J16; footprint Connector_PinHeader_2.54mm:PinHeader_1x04_P2.54mm_Vertical -> Connector_JST:JST_EH_B4B-EH-A_1x04_P2.50mm_Vertical
- J9: renamed from J6; footprint Connector_PinHeader_2.54mm:PinHeader_1x03_P2.54mm_Vertical -> Connector_JST:JST_EH_B3B-EH-A_1x03_P2.50mm_Vertical
Connections:
- net labels added: Input1BTN_SCK, PowerLEDGND
- net labels removed: Input1Btn, PowerLED, SCK
- wire segments 221 -> 228

Commit message: Update preamp scheme: add led resistors
Parts:
- added R1, R2, R3, R4, R5, R6, R7: 1k, Resistor_THT:R_Axial_DIN0309_L9.0mm_D3.2mm_P12.70mm_Horizontal, symbol Device:R
- R10: renamed from R3; footprint Resistor_THT:R_Axial_DIN0207_L6.3mm_D2.5mm_P10.16mm_Horizontal -> Resistor_THT:R_Axial_DIN0309_L9.0mm_D3.2mm_P12.70mm_Horizontal
- R11: renamed from R4; footprint Resistor_THT:R_Axial_DIN0207_L6.3mm_D2.5mm_P10.16mm_Horizontal -> Resistor_THT:R_Axial_DIN0309_L9.0mm_D3.2mm_P12.70mm_Horizontal
- R12: renamed from R5; footprint Resistor_THT:R_Axial_DIN0207_L6.3mm_D2.5mm_P10.16mm_Horizontal -> Resistor_THT:R_Axial_DIN0309_L9.0mm_D3.2mm_P12.70mm_Horizontal
- R13: renamed from R6; footprint Resistor_THT:R_Axial_DIN0207_L6.3mm_D2.5mm_P10.16mm_Horizontal -> Resistor_THT:R_Axial_DIN0309_L9.0mm_D3.2mm_P12.70mm_Horizontal
- R14: renamed from R7; footprint Resistor_THT:R_Axial_DIN0207_L6.3mm_D2.5mm_P10.16mm_Horizontal -> Resistor_THT:R_Axial_DIN0309_L9.0mm_D3.2mm_P12.70mm_Horizontal
- R8: renamed from R1; footprint Resistor_THT:R_Axial_DIN0207_L6.3mm_D2.5mm_P10.16mm_Horizontal -> Resistor_THT:R_Axial_DIN0309_L9.0mm_D3.2mm_P12.70mm_Horizontal
- R9: renamed from R2; footprint Resistor_THT:R_Axial_DIN0207_L6.3mm_D2.5mm_P10.16mm_Horizontal -> Resistor_THT:R_Axial_DIN0309_L9.0mm_D3.2mm_P12.70mm_Horizontal
- renumbered J2 to J1, J3 to J2, J4 to J3, J5 to J4, J6 to J5, J7 to J6, J8 to J7, J1 to J8
Connections:
- wire segments 228 -> 242

Commit message: Update preamp scheme: add +5V power
Parts:
- removed J15: CONN_01X02, Connector_JST:JST_EH_B3B-EH-A_1x03_P2.50mm_Vertical, symbol Connector_Generic:Conn_01x02
- added C13, C15: 100uF, Capacitor_THT:CP_Radial_D5.0mm_P2.50mm, symbol Device:CP_Small
- added C18: 100nF, Capacitor_THT:C_Rect_L9.0mm_W2.5mm_P7.50mm_MKT, symbol Device:C_Small
- added C8: 0.33uF, Capacitor_THT:C_Rect_L9.0mm_W2.5mm_P7.50mm_MKT, symbol Device:C_Small
- added J15, J16: CONN_01X03, Connector_JST:JST_EH_B3B-EH-A_1x03_P2.50mm_Vertical, symbol Connector_Generic:Conn_01x03
- added U3: LM7805, Package_TO_SOT_THT:TO-220-3_Horizontal_TabDown, symbol Regulator_Linear:LM78L05_TO92
- renumbered C9 to C10, C10 to C11, C11 to C12, C12 to C14, C13 to C16, C14 to C17, C15 to C19, C16 to C20, C17 to C21, C18 to C22, C19 to C23, C20 to C24, C21 to C25, C22 to C26, C23 to C27, C8 to C9, J16 to J17, U3 to U4, U4 to U5
Connections:
- net labels added: +5V
- wire segments 242 -> 269
