File: examples/preamp/cad/preamp.sch (KiCad schematic (older format))
At the start: 68 parts, among them CON1 AVR-ISP-10, J1 Conn_01x04, J10 Conn_01x04, J11 CONN_01X03, J12 Conn_01x03, J13 Conn_01x03, J14 Conn_01x03, J15 CONN_01X03, J16 CONN_01X03, J17 CONN_01X03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

Commit message: Update preamp pcb
Connections:
- wire segments 269 -> 270

Commit message: Preamp PCB update
Parts:
- added C28: 100uF, Capacitor_THT:CP_Radial_D5.0mm_P2.50mm, symbol Device:CP_Small
Connections:
- wire segments 270 -> 273
Changed lines of the file:
@@
 VCC
-Wire Wire Line
-	7750 6800 7950 6800
 Wire Wire Line
 	7750 6900 7950 6900
@@
 $EndComp
 $Comp
-L power:GND #PWR?
+L power:GND #PWR033
 U 1 1 5E2554ED
 P 5775 7875
-F 0 "#PWR?" H 5775 7625 50  0001 C CNN
+F 0 "#PWR033" H 5775 7625 50  0001 C CNN
 F 1 "GND" H 5775 7725 50  0000 C CNN
 F 2 "" H 5775 7875 50  0001 C CNN
@@
 Wire Wire Line
 	5775 7800 5775 7875
+Connection ~ 5775 7800
+$Comp
+L Device:CP_Small C28
+U 1 1 5E57F603
+P 7525 6900
+F 0 "C28" H 7535 6970 50  0000 L CNN
+F 1 "100uF" H 7535 6820 50  0000 L CNN
+F 2 "Capacitor_THT:CP_Radial_D5.0mm_P2.50mm" H 7525 6900 50  0001 C CNN
+F 3 "~" H 7525 6900 50  0001 C CNN
+	1    7525 6900
+	1    0    0    -1
+$EndComp
+Wire Wire Line
+	7525 6800 7950 6800
+Wire Wire Line
+	7525 7000 7650 7000
+Wire Wire Line
+	7650 7000 7650 6900
+Wire Wire Line
+	7650 6900 7750 6900
 Wire Bus Line
 	6200 1900 8400 1900
@@
 Wire Bus Line
 	6200 1900 6200 10150
-Connection ~ 5775 7800
+Connection ~ 7750 6900
 $EndSCHEMATC

Commit message: preamp: fix R value
Parts:
- R9: value 10k -> 47k
Changed lines of the file:
@@
 EESchema Schematic File Version 4
-LIBS:preamp-cache
 EELAYER 30 0
 EELAYER END
@@
 P 6700 8550
 F 0 "R9" V 6780 8550 50  0000 C CNN
-F 1 "10k" V 6700 8550 50  0000 C CNN
+F 1 "47k" V 6700 8550 50  0000 C CNN
 F 2 "Resistor_THT:R_Axial_DIN0309_L9.0mm_D3.2mm_P12.70mm_Horizontal" V 6630 8550 50  0001 C CNN
 F 3 "~" H 6700 8550 50  0001 C CNN
@@
 Wire Wire Line
 	7650 6900 7750 6900
+Connection ~ 7750 6900
 Wire Bus Line
 	6200 1900 8400 1900
@@
 Wire Bus Line
 	6200 1900 6200 10150
-Connection ~ 7750 6900
 $EndSCHEMATC
